File: Hardware/Kicad projects/MainBoard/mainPCB/_autosave-mainPCB.kicad_sch (KiCad schematic)
At the start: 52 parts, among them J1 USB_C_Receptacle_USB2.0, J2 Conn_01x18, J3 +VIN-, J4 Micro_SD_Card, J5 ENC_L, J6 ENC_R, J9 Conn_01x03, SW1 SW_DPDT_x2, U1 TB6612FNG, U10 TB6612FNG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

Commit message: hiu
Parts:
- removed MotorL1, MotorR1: Conn_01x02, Connector_JST:JST_ZH_B2B-ZR_1x02_P1.50mm_Vertical, symbol Connector_Generic:Conn_01x02
Connections:
- net at MotorL1.1 (Pin_1), U1.1 (AO1), U1.11 (BO1)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: now also U9.1 (AO1), U9.11 (BO1), U9.12 (BO1), U9.2 (AO1)
- net at MotorL1.2 (Pin_2), U1.5 (AO2), U1.6 (AO2)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: now also U9.5 (AO2), U9.6 (AO2), U9.7 (BO2), U9.8 (BO2)
- net at U10.1 (AO1), U10.11 (BO1), U10.12 (BO1)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: now also MotorR1.1 (Pin_1), U3.1 (AO1), U3.11 (BO1), U3.12 (BO1), U3.2 (AO1)
- net at U10.5 (AO2), U10.6 (AO2), U10.7 (BO2)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: now also MotorR1.2 (Pin_2), U3.5 (AO2), U3.6 (AO2), U3.7 (BO2), U3.8 (BO2)
Other:
- moved on the sheet: MotorR1
