File: Hardware/Kicad projects/MainBoard/mainPCB/mainPCB.kicad_sch (KiCad schematic)
At the start: 50 parts, among them J1 USB_C_Receptacle_USB2.0, J2 Conn_01x18, J3 +VIN-, J4 Micro_SD_Card, J5 ENC_L, J6 ENC_R, J9 Conn_01x03, SW1 SW_DPDT_x2, U1 TB6612FNG, U10 TB6612FNG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

Commit message: fefewfe
fefef
Parts:
- removed J2: Conn_01x18, Connector_FFC-FPC:Hirose_FH12-18S-0.5SH_1x18-1MP_P0.50mm_Horizontal, symbol Connector_Generic:Conn_01x18
- removed J3: +VIN-, Connector_PinHeader_2.54mm:PinHeader_1x02_P2.54mm_Vertical, symbol Connector_Generic:Conn_01x02
- added D3, D4, D5, D6: BLUE, LED_SMD:LED_0603_1608Metric, symbol Device:LED_Small
- added J2: Conn_01x08, Connector_FFC-FPC:Hirose_FH12-8S-0.5SH_1x08-1MP_P0.50mm_Horizontal, symbol Connector_Generic:Conn_01x08
- added J7: Conn_01x04, symbol Connector_Generic:Conn_01x04
- added R10, R11, R12, R9: 510R, Resistor_SMD:R_0603_1608Metric, symbol Device:R
- added SW2: SW_SPST, Button_Switch_SMD:SW_SPST_CK_RS282G05A3, symbol Switch:SW_SPST
- added SW3: SW_DPDT_x2, Button_Switch_SMD:SW_SPDT_PCM12, symbol Switch:SW_DPDT_x2
- added U5: W25Q32JVSS, Package_SO:SOIC-8_5.23x5.23mm_P1.27mm, symbol Memory_Flash:W25Q32JVSS
- renumbered J9 to Converter
Connections:
- net Sensor12 is gone; now on net ENC_R_I: U2.21 (PA7)
- net +3.3V: now also J2.1 (Pin_1)
- net +3V3: now also SW3.3 (C)
- net 2S FROM LIPO: now also J7.2 (Pin_2)
- net ENC_L_I: now also U2.58 (PB5)
- net GND: now also D3.1 (K), D4.1 (K), D5.1 (K), D6.1 (K), J2.8 (Pin_8), J7.4 (Pin_4), SW2.1 (A), SW3.1 (A)
- net NRST: now also SW2.2 (B)
- net VDC: now also J7.1 (Pin_1)
- net Sensor1 renamed S3
- net S3: now also J2.5 (Pin_5)
- net Sensor10 renamed S0
- net S0: now also J2.2 (Pin_2)
- net Sensor11 renamed Function
- net Function: now also SW3.2 (B)
- net Sensor2 renamed ADC
- net ADC: now also J2.6 (Pin_6)
- net Sensor3 renamed Enable
- net Enable: now also J2.7 (Pin_7)
- net Sensor4 renamed LED_6
- net LED_6: now also R12.2
- net Sensor5 renamed LED_5
- net LED_5: now also R11.2
- net Sensor6 renamed LED_4
- net LED_4: now also R10.2
- net Sensor7 renamed LED_3
- net LED_3: now also R9.2
- net Sensor8 renamed S2
- net S2: now also J2.4 (Pin_4)
- net Sensor9 renamed S1
- net S1: now also J2.3 (Pin_3)
- new net: D6.2 (A), R12.1
- new net: D5.2 (A), R11.1
- new net: D4.2 (A), R10.1
- new net: D3.2 (A), R9.1
- new net 1S FROM LIPO: J7.3 (Pin_3)
- no-connect marks 17 -> 15
Other:
- note added: "2x TB6612FNG Motor Driver L 4A"
- note added: "2x TB6612FNG Motor Driver R 4A"
- note added: "FAULHABER SR1024 6V motors 12t on motor 0.3M"
- note added: "FaulHaber Encoders IEB 128"
- note added: "Function switch"
- note added: "LiPo 12,6V JST connector"
- note removed: "LiPo 7,4V JST connector"
- note removed: "Regulated footprint for Encoders"
- note removed: "TB6612FNG Motor Driver L"
- note removed: "TB6612FNG Motor Driver R"
- moved on the sheet: C8, Converter, IMU1, R6, R7, SW1A
